Commit message: second commit

File: robot_model/urdf/wheel.urdf.xacro (robot description, xacro)
@@ -2,11 +2,11 @@
 <robot name="wheel" xmlns:xacro="http://www.ros.org/wiki/xacro">
     <xacro:property name="M_PI" value="3.1415926535897931" />
-    <xacro:property name="wheel_radius" value="0.05" />
-    <xacro:property name="wheel_height" value="0.045" />
+    <xacro:property name="wheel_radius" value="0.0475" /> <!-- m -->
+    <xacro:property name="wheel_depth" value="0.015" />
     <xacro:property name="wheel_mass" value="2.5" /> <!-- in kg-->
     <!-- translate form origin to wheel coordinate -->
-    <xacro:property name="base_x_base_link_to_wheel_origin" value="0.2" />
-    <xacro:property name="base_y_base_link_to_wheel_origin" value="0.1" />
-    <xacro:property name="base_z_base_link_to_wheel_origin" value="-0.075" />
+    <xacro:property name="base_x_base_link_to_wheel_origin" value="0.0" />
+    <xacro:property name="base_y_base_link_to_wheel_origin" value="0.16" />
+    <xacro:property name="base_z_base_link_to_wheel_origin" value="0.0" />
     <xacro:macro name="cylinder_inertia" params="m r h">
     <inertia  ixx="${m*(3*r*r+h*h)/12}" ixy = "0" ixz = "0"
@@ -15,11 +15,11 @@
     </xacro:macro>
     <!-- fb: front back, lr: left right, translateX, Y: + -, flipY: rotate along Y -->
-    <xacro:macro name="wheel" params="fb lr parent translateX translateY flipY">
+    <xacro:macro name="wheel" params="lr parent translateX translateY flipY">
         <!-- joint -->
-        <link name="${fb}_${lr}_wheel">
+        <link name="${lr}_wheel">
             <visual>
                 <origin xyz="0 0 0" rpy="${flipY*M_PI/2} 0  0 " />
                 <geometry>
-                    <cylinder length="${wheel_height}" radius="${wheel_radius}" />
+                    <cylinder length="${wheel_depth}" radius="${wheel_radius}" />
                 </geometry>
                 <material name="Black" />
@@ -28,5 +28,5 @@
                 <origin xyz="0 0 0" rpy="${flipY*M_PI/2} 0 0 " />
                 <geometry>
-                    <cylinder length="${wheel_height}" radius="${wheel_radius}" />
+                    <cylinder length="${wheel_depth}" radius="${wheel_radius}" />
                 </geometry>
             </collision>
@@ -34,9 +34,9 @@
                 <mass value="${wheel_mass}" />
                 <origin xyz="0 0 0" />
-                <cylinder_inertia  m="${wheel_mass}" r="${wheel_radius}" h="${wheel_height}" />
+                <cylinder_inertia  m="${wheel_mass}" r="${wheel_radius}" h="${wheel_depth}" />
             </inertial>
         </link>
         <!-- gazebo -->
-        <gazebo reference="${fb}_${lr}_wheel">
+        <gazebo reference="${lr}_wheel">
             <mu1 value="1.0"/>
             <mu2 value="1.0"/>
@@ -48,8 +48,8 @@
         </gazebo>
         <!-- joint -->
-        <joint name="${fb}_${lr}_wheel_joint" type="continuous">
+        <joint name="${lr}_wheel_joint" type="continuous">
             <parent link="${parent}"/>
-            <child link="${fb}_${lr}_wheel"/>
-            <origin xyz="${translateX * (base_x_base_link_to_wheel_origin - wheel_radius)} ${translateY * (base_y_base_link_to_wheel_origin + wheel_height/2)} ${base_z_base_link_to_wheel_origin}" rpy="0 0 0" />
+            <child link="${lr}_wheel"/>
+            <origin xyz="${translateX * (base_x_base_link_to_wheel_origin)} ${translateY * (base_y_base_link_to_wheel_origin + wheel_depth/2)} ${base_z_base_link_to_wheel_origin}" rpy="0 0 0" />
             <axis xyz="0 1 0" rpy="0 0 0" />
             <limit effort="100" velocity="100"/>
@@ -57,8 +57,8 @@
         </joint>
         <!-- Transmission wheel -->
-        <transmission name="${fb}_${lr}_wheel_joint_trans">
+        <transmission name="${lr}_wheel_joint_trans">
             <type>transmission_interface/SimpleTransmission</type>
-            <joint name="${fb}_${lr}_wheel_joint" />
-            <actuator name="${fb}_${lr}_wheel_joint_motor">
+            <joint name="${lr}_wheel_joint" />
+            <actuator name="${lr}_wheel_joint_motor">
                 <hardwareInterface>EffortJointInterface</hardwareInterface>
                 <mechanicalReduction>1</mechanicalReduction>
